File: pcb_matrix8/pcb_matrix8.kicad_pcb (KiCad board)
At the start: 2 copper layers, 525 x 62.5 mm, 18 parts, among them J1 DIN 1, J10 DOUT 6, J11 DOUT 7, J12 DOUT 8, J13 DIN 4, J14 DIN 5, J15 DIN 6, J16 DIN 7, J17 DIN 8, J18 OUT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

Commit message: pcb 2
Routing:
- net +5V: track 450.3 -> 471.6 mm
- net GND: track 30.8 -> 32.8 mm
